File: WiFiRelay.kicad_pcb (KiCad board)
At the start: 2 copper layers, 20 parts, among them J1 Serial, J2 Conn_01x04, K1 TRA2-L-3VDC-S-Z, Q1 IRLML0030, SW1 SW_Push, SW2 SW_Push, U1 ESP-12E

Commit message: release
Parts:
- removed J1: Serial, Connector_PinHeader_2.54mm:PinHeader_1x04_P2.54mm_Vertical
- removed SW1: SW_Push, Resistor_SMD:R_0805_2012Metric_Pad1.20x1.40mm_HandSolder
- added IO0: SW_Push, Resistor_SMD:R_0805_2012Metric_Pad1.20x1.40mm_HandSolder, F.Cu at (142.0, 119.2)
- added REF**: Symbol_HighVoltage_Triangle_6x6mm_Copper, Symbol:Symbol_HighVoltage_Triangle_6x6mm_Copper, F.Cu at (77.0, 90.5)
- added REF**: Symbol_HighVoltage_Triangle_6x6mm_Copper, Symbol:Symbol_HighVoltage_Triangle_6x6mm_Copper, B.Cu at (91.0, 98.0)
- added UART1: Serial, Connector_PinHeader_2.54mm:PinHeader_1x04_P2.54mm_Vertical, F.Cu at (141.8, 125.2)
- SW2: footprint Connector_PinHeader_2.54mm:PinHeader_1x04_P2.54mm_Vertical -> Connector_PinHeader_2.54mm:PinHeader_1x02_P2.54mm_Vertical
- moved C1 69.4 mm to (113.2, 116.0), turned to 90 degrees
- moved C2 64.9 mm to (116.2, 116.0), turned to 90 degrees
- moved SW2 63.9 mm to (136.8, 118.0), turned to -90 degrees
- moved D2 50.8 mm to (121.0, 105.7), turned to -90 degrees
- moved R6 47.4 mm to (119.2, 116.0), turned to 90 degrees
- moved R3 35.7 mm to (127.2, 123.0), turned to 180 degrees
- moved R2 32.3 mm to (121.8, 101.0)
- moved R1 32.1 mm to (121.8, 97.0)
- moved U1 9.82 mm to (134.5, 100.5), turned to 0 degrees
- moved R4 5.00 mm to (127.0, 117.5), turned to 90 degrees
- moved R5 0.25 mm to (127.2, 126.0)
Connections:
- K1 pad 18: Net-(F1-Pad2) -> /LOAD
- K1 pad 27: /LOAD -> Net-(F1-Pad2)
- R6 pad 1: Net-(U1-GPIO10) -> Net-(U1-GPIO16)
- U1 pad 12: Net-(U1-GPIO10) -> unconnected-(U1-GPIO10-Pad12)
- U1 pad 4: unconnected-(U1-GPIO16-Pad4) -> Net-(U1-GPIO16)
Routing:
- net +3V3: track 0.00 -> 93.1 mm, vias 0 -> 1
- net GND: track 0.00 -> 43.4 mm, vias 0 -> 1
- net Net-(U1-GPIO1/TXD): track 0.00 -> 31.8 mm, vias 0 -> 1
- net Net-(U1-GPIO0): track 0.00 -> 31.3 mm
- net Net-(U1-GPIO3/RXD): track 0.00 -> 28.9 mm, vias 0 -> 1
- net Net-(U1-GPIO16): track 0.00 -> 20.3 mm
- net /LOAD: track 26.3 -> 9.50 mm
- net Net-(D1-A): track 0.00 -> 12.7 mm
- net Net-(Q1-G): track 0.00 -> 11.9 mm
- net /RELAY: track 0.00 -> 9.80 mm
- net Net-(D2-A): track 0.00 -> 6.91 mm
- net Net-(U1-GPIO9): track 0.00 -> 5.83 mm
- net Net-(U1-~{RST}): track 0.00 -> 3.62 mm
- net Net-(U1-EN): track 0.00 -> 3.62 mm
- added copper zone on F.Cu, net GND
Other:
- board outline added: 80 x 45 mm
- board text added: "WiFi Relay V1.0"

Commit message: fix pins
Parts:
- removed REF** (x2): Symbol_HighVoltage_Triangle_6x6mm_Copper, Symbol:Symbol_HighVoltage_Triangle_6x6mm_Copper
- added R7: 10k, Resistor_SMD:R_1206_3216Metric_Pad1.30x1.75mm_HandSolder, F.Cu at (130.0, 117.5)
- D1: value D -> 1N4007
- moved SW2 2.61 mm to (134.2, 118.0), turned to 90 degrees
- moved IO0 0.25 mm to (142.0, 119.0)
Connections:
- SW2 pad 1: GND -> Net-(U1-GPIO4)
- SW2 pad 2: Net-(U1-GPIO9) -> GND
- U1 pad 11: Net-(U1-GPIO9) -> unconnected-(U1-GPIO9-Pad11)
- U1 pad 16: GND -> Net-(U1-GPIO15)
- U1 pad 19: unconnected-(U1-GPIO4-Pad19) -> Net-(U1-GPIO4)
Routing:
- net Net-(U1-GPIO15): track 0.00 -> 25.4 mm
- net Net-(U1-GPIO4): track 0.00 -> 20.1 mm
- net Net-(U1-GPIO9): track 5.83 -> 0.00 mm
- net GND: track 43.4 -> 45.8 mm
- net Net-(U1-GPIO0): track 31.3 -> 31.8 mm
