File: WiFiRelay.kicad_sch (KiCad schematic)
At the start: 20 parts, among them J1 Serial, J2 Conn_01x04, K1 TRA2-L-3VDC-S-Z, Q1 IRLML0030, SW1 SW_Push, SW2 SW_Push, U1 ESP-12E

Commit message: release
Parts:
- C1: Price (none) -> 24; Purchase-URL (none) -> https://www.chipdip.ru/product/grm31cr61a106k
- C2: Price (none) -> 8
- D1: value D -> 1N4007; Price (none) -> 0,8; Purchase-URL (none) -> https://aliexpress.ru/item/32731035430.html?sku_id=12000018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
- D2: Price (none) -> 19; Purchase-URL (none) -> https://www.chipdip.ru/product/l-1154gt
- F1: Price (none) -> 44; Purchase-URL (none) -> https://aliexpress.ru/item/1005002933092692.html?sku_id=120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
- F2: Price (none) -> 39; Purchase-URL (none) -> https://www.chipdip.ru/product/mf02s84-1000-1
- J2: Price None -> 33; Purchase-URL https://www.snapeda.com/api/url_track_click_mouser/?unipart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 -> https://www.chipdip.ru/product/300-041-12
- K1: Price (none) -> 88; Purchase-URL (none) -> https://www.chipdip.ru/product0/8025423609
- PS1: Price (none) -> 170
- Q1: Price (none) -> 19; Purchase-URL (none) -> https://www.chipdip.ru/product0/8017689792
- R1, R2, R3, R4, R5, R6: Price (none) -> 0,4
- SW2: footprint Connector_PinHeader_2.54mm:PinHeader_1x04_P2.54mm_Vertical -> Connector_PinHeader_2.54mm:PinHeader_1x02_P2.54mm_Vertical; Price (none) -> 33
- U1: Price (none) -> 100
- renumbered SW1 to IO0, J1 to UART1
Connections:
- net LOAD: now also K1.18; no longer K1.27
- net at U1.12 (GPIO10): no longer R6.1
- net at U1.4 (GPIO16): now also R6.1
- net at F1.2: now also K1.27; no longer K1.18
Other:
- moved on the sheet: D1, D2, F1, R6

Commit message: fix pins
Parts:
- added R7: 10k, Resistor_SMD:R_1206_3216Metric_Pad1.30x1.75mm_HandSolder, symbol Device:R
Connections:
- net GND: now also SW2.2, R7.2; no longer SW2.1, U1.16 (GPIO15)
- net at U1.11 (GPIO9): no longer SW2.2
- net at U1.19 (GPIO4): now also SW2.1
- new net: R7.1, U1.16 (GPIO15)
Other:
- moved on the sheet: SW2, UART1
Changed lines of the file:
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@@
 	(wire
 		(pts
-			(xy 120.65 101.6) (xy 123.19 101.6)
-		)
-		(stroke
-			(width 0)
-			(type default)
-		)
-	)
-	(wire
-		(pts
 			(xy 60.96 57.15) (xy 60.96 60.96)
 		)
@@
 	(wire
 		(pts
-			(xy 107.95 101.6) (xy 110.49 101.6)
+			(xy 198.12 101.6) (xy 195.58 101.6)
 		)
 		(stroke
@@
 	(wire
 		(pts
+			(xy 184.15 101.6) (xy 185.42 101.6)
+		)
+		(stroke
+			(width 0)
+			(type default)
+		)
+	)
+	(wire
+		(pts
 			(xy 48.26 66.04) (xy 50.8 66.04)
 		)
@@
 	(wire
 		(pts
+			(xy 165.1 104.14) (xy 170.18 104.14)
+		)
+		(stroke
+			(width 0)
+			(type default)
+		)
+	)
+	(wire
+		(pts
 			(xy 158.75 83.82) (xy 153.67 83.82)
 		)
@@
 	(wire
 		(pts
-			(xy 158.75 87.63) (xy 168.91 87.63)
+			(xy 158.75 87.63) (xy 172.72 87.63)
 		)
 		(stroke
@@
 	(wire
 		(pts
+			(xy 161.29 91.44) (xy 161.29 96.52)
+		)
+		(stroke
+			(width 0)
+			(type default)
+		)
+	)
+	(wire
+		(pts
 			(xy 153.67 106.68) (xy 157.48 106.68)
 		)
@@
 	(wire
 		(pts
+			(xy 153.67 91.44) (xy 161.29 91.44)
+		)
+		(stroke
+			(width 0)
+			(type default)
+		)
+	)
+	(wire
+		(pts
 			(xy 109.22 81.28) (xy 109.22 74.93)
 		)
@@
 	(wire
 		(pts
-			(xy 153.67 104.14) (xy 156.21 104.14)
+			(xy 153.67 104.14) (xy 157.48 104.14)
 		)
 		(stroke
@@
 	(wire
 		(pts
-			(xy 158.75 85.09) (xy 168.91 85.09)
+			(xy 184.15 96.52) (xy 184.15 101.6)
+		)
+		(stroke
+			(width 0)
+			(type default)
+		)
+	)
+	(wire
+		(pts
+			(xy 158.75 85.09) (xy 172.72 85.09)
 		)
 		(stroke
@@
 		)
 	)
+	(wire
+		(pts
+			(xy 161.29 96.52) (xy 184.15 96.52)
+		)
+		(stroke
+			(width 0)
+			(type default)
+		)
+	)
 	(label "LOAD"
 		(at 62.23 113.03 270)
@@
 	(symbol
 		(lib_id "Switch:SW_Push")
-		(at 115.57 101.6 0)
+		(at 190.5 101.6 0)
 		(unit 1)
 		(exclude_from_sim no)
@@
 		(fields_autoplaced yes)
 		(property "Reference" "SW2"
-			(at 115.57 93.98 0)
+			(at 190.5 93.98 0)
 			(effects
 				(font
@@
 		)
 		(property "Value" "SW_Push"
-			(at 115.57 96.52 0)
+			(at 190.5 96.52 0)
 			(effects
 				(font
@@
 		)
 		(property "Footprint" "Connector_PinHeader_2.54mm:PinHeader_1x02_P2.54mm_Vertical"
-			(at 115.57 96.52 0)
+			(at 190.5 96.52 0)
 			(effects
 				(font
@@
 		)
 		(property "Datasheet" "~"
-			(at 115.57 96.52 0)
+			(at 190.5 96.52 0)
 			(effects
 				(font
@@
 		)
 		(property "Description" "Push button switch, generic, two pins"
-			(at 115.57 101.6 0)
+			(at 190.5 101.6 0)
 			(effects
 				(font
@@
 		)
 		(property "Price" "33"
-			(at 115.57 101.6 0)
+			(at 190.5 101.6 0)
 			(effects
 				(font
@@
 	(symbol
 		(lib_id "power:+3V3")
-		(at 168.91 90.17 90)
+		(at 172.72 90.17 90)
 		(unit 1)
 		(exclude_from_sim no)
@@
 		(fields_autoplaced yes)
 		(property "Reference" "#PWR013"
-			(at 172.72 90.17 0)
+			(at 176.53 90.17 0)
 			(effects
 				(font
@@
 		)
 		(property "Value" "+3V3"
-			(at 165.1 90.1699 90)
+			(at 168.91 90.1699 90)
 			(effects
 				(font
@@
 		)
 		(property "Footprint" ""
-			(at 168.91 90.17 0)
+			(at 172.72 90.17 0)
 			(effects
 				(font
@@
 		)
 		(property "Datasheet" ""
-			(at 168.91 90.17 0)
+			(at 172.72 90.17 0)
 			(effects
 				(font
@@
 		)
 		(property "Description" "Power symbol creates a global label with name \"+3V3\""
-			(at 168.91 90.17 0)
+			(at 172.72 90.17 0)
 			(effects
 				(font
@@
 	(symbol
 		(lib_id "power:GND")
-		(at 156.21 104.14 90)
+		(at 170.18 104.14 90)
 		(unit 1)
 		(exclude_from_sim no)
@@
 		(fields_autoplaced yes)
 		(property "Reference" "#PWR06"
-			(at 162.56 104.14 0)
+			(at 176.53 104.14 0)
 			(effects
 				(font
@@
 		)
 		(property "Value" "GND"
-			(at 160.02 104.1399 90)
+			(at 173.99 104.1399 90)
 			(effects
 				(font
@@
 		)
 		(property "Footprint" ""
-			(at 156.21 104.14 0)
+			(at 170.18 104.14 0)
 			(effects
 				(font
@@
 		)
 		(property "Datasheet" ""
-			(at 156.21 104.14 0)
+			(at 170.18 104.14 0)
 			(effects
 				(font
@@
 		)
 		(property "Description" "Power symbol creates a global label with name \"GND\" , ground"
-			(at 156.21 104.14 0)
+			(at 170.18 104.14 0)
 			(effects
 				(font
@@
 	(symbol
 		(lib_id "power:GND")
-		(at 107.95 101.6 270)
+		(at 198.12 101.6 90)
 		(unit 1)
 		(exclude_from_sim no)
@@
 		(fields_autoplaced yes)
 		(property "Reference" "#PWR014"
-			(at 101.6 101.6 0)
+			(at 204.47 101.6 0)
 			(effects
 				(font
@@
 		)
 		(property "Value" "GND"
-			(at 104.14 101.5999 90)
+			(at 201.93 101.6001 90)
 			(effects
 				(font
@@
 		)
 		(property "Footprint" ""
-			(at 107.95 101.6 0)
+			(at 198.12 101.6 0)
 			(effects
 				(font
@@
 		)
 		(property "Datasheet" ""
-			(at 107.95 101.6 0)
+			(at 198.12 101.6 0)
 			(effects
 				(font
@@
 		)
 		(property "Description" "Power symbol creates a global label with name \"GND\" , ground"
-			(at 107.95 101.6 0)
+			(at 198.12 101.6 0)
 			(effects
 				(font
@@
 	)
 	(symbol
+		(lib_id "Device:R")
+		(at 161.29 104.14 90)
+		(unit 1)
+		(exclude_from_sim no)
+		(in_bom yes)
+		(on_board yes)
+		(dnp no)
+		(property "Reference" "R7"
+			(at 161.29 101.854 90)
+			(effects
+				(font
+					(size 1.27 1.27)
+				)
+			)
+		)
+		(property "Value" "10k"
+			(at 161.29 106.172 90)
+			(effects
+				(font
+					(size 1.27 1.27)
+				)
+			)
+		)
+		(property "Footprint" "Resistor_SMD:R_1206_3216Metric_Pad1.30x1.75mm_HandSolder"
+			(at 161.29 105.918 90)
+			(effects
+				(font
+					(size 1.27 1.27)
+				)
+				(hide yes)
+			)
+		)
+		(property "Datasheet" "~"
+			(at 161.29 104.14 0)
+			(effects
+				(font
+					(size 1.27 1.27)
+				)
+				(hide yes)
+			)
+		)
+		(property "Description" "Resistor"
+			(at 161.29 104.14 0)
+			(effects
+				(font
+					(size 1.27 1.27)
+				)
+				(hide yes)
+			)
+		)
+		(property "Price" "0,4"
+			(at 161.29 104.14 0)
+			(effects
+				(font
+					(size 1.27 1.27)
+				)
+				(hide yes)
+			)
+		)
+		(pin "2"
+		)
+		(pin "1"
+		)
+		(instances
+			(project "WiFiRelay"
+				(path "/456f6305-4497-43ef-94cc-8a7589663bc4"
+					(reference "R7")
+					(unit 1)
+				)
+			)
+		)
+	)
+	(symbol
 		(lib_id "Converter_ACDC:HLK-PM03")
 		(at 170.18 31.75 0)
@@
 	(symbol
 		(lib_id "Connector_Generic:Conn_01x04")
-		(at 173.99 87.63 0)
+		(at 177.8 87.63 0)
 		(unit 1)
 		(exclude_from_sim no)
@@
 		(fields_autoplaced yes)
 		(property "Reference" "UART1"
-			(at 176.53 87.6299 0)
+			(at 180.34 87.6299 0)
 			(effects
 				(font
@@
 		)
 		(property "Value" "Serial"
-			(at 176.53 90.1699 0)
+			(at 180.34 90.1699 0)
 			(effects
 				(font
@@
 		)
 		(property "Footprint" "Connector_PinHeader_2.54mm:PinHeader_1x04_P2.54mm_Vertical"
-			(at 173.99 87.63 0)
+			(at 177.8 87.63 0)
 			(effects
 				(font
@@
 		)
 		(property "Datasheet" "~"
-			(at 173.99 87.63 0)
+			(at 177.8 87.63 0)
 			(effects
 				(font
@@
 		)
 		(property "Description" "Generic connector, single row, 01x04, script generated (kicad-library-utils/schlib/autogen/connector/)"
-			(at 173.99 87.63 0)
+			(at 177.8 87.63 0)
 			(effects
 				(font
@@
 	(symbol
 		(lib_id "power:GND")
-		(at 168.91 92.71 270)
+		(at 172.72 92.71 270)
 		(unit 1)
 		(exclude_from_sim no)
@@
 		(fields_autoplaced yes)
 		(property "Reference" "#PWR012"
-			(at 162.56 92.71 0)
+			(at 166.37 92.71 0)
 			(effects
 				(font
@@
 		)
 		(property "Value" "GND"
-			(at 165.1 92.7099 90)
+			(at 168.91 92.7099 90)
 			(effects
 				(font
@@
 		)
 		(property "Footprint" ""
-			(at 168.91 92.71 0)
+			(at 172.72 92.71 0)
 			(effects
 				(font
@@
 		)
 		(property "Datasheet" ""
-			(at 168.91 92.71 0)
+			(at 172.72 92.71 0)
 			(effects
 				(font
@@
 		)
 		(property "Description" "Power symbol creates a global label with name \"GND\" , ground"
-			(at 168.91 92.71 0)
+			(at 172.72 92.71 0)
 			(effects
 				(font
